File: Hardware/Production/SparkFun_Tsunami_Qwiic-Panel_v22.brd (EAGLE design)
At the start: 257.3 x 169.4 mm, 1956 parts, among them J1 VDC-IN, J10 TRIG2, J11 TRIG1, J12 3.3VA, J14 AUDIO I/O, J15 MIDI, J16 USB-C, J17 AGND, J19 3.3V, J2 GND-IN, J20 TRIG2, J21 TRIG1, J22 MIDI, J23 DEBUG, J24 PLAYING, J25 VDC-IN, J26 GND-IN, J27 USB-C, J28 QWIIC, J29 AGND, J3 DEBUG, J32 CORTEX_JTAG_DEBUG_PTH_NS, J33 AUDIO I/O, J34 3.3VA, J35 3.3V, J36 TRIG2, J37 TRIG1, J38 MIDI, J39 DEBUG, J4 QWIIC, J40 PLAYING, J41 VDC-IN, J42 GND-IN, J43 USB-C, J44 QWIIC, J45 AGND, J48 CORTEX_JTAG_DEBUG_PTH_NS, J49 AUDIO I/O, J5 AUDIO I/O, J50 3.3VA, J51 3.3V, J52 TRIG2, J53 TRIG1, J54 MIDI, J55 DEBUG, J56 PLAYING, J57 VDC-IN, J58 GND-IN, J59 USB-C, J6 3.3VA, J60 QWIIC, J61 AGND, J64 CORTEX_JTAG_DEBUG_PTH_NS, J65 AUDIO I/O, J66 3.3VA, J67 3.3V, J68 TRIG2, J69 TRIG1, J7 3.3V, J70 MIDI, J71 DEBUG, J72 PLAYING, J73 VDC-IN, J74 GND-IN, J75 USB-C, J76 QWIIC, J77 AGND, J8 PLAYING, J80 CORTEX_JTAG_DEBUG_PTH_NS, J81 AUDIO I/O, J82 3.3VA, J83 3.3V, J84 TRIG2, J85 TRIG1, J86 MIDI, J87 DEBUG, J88 PLAYING, J89 VDC-IN, J9 CORTEX_JTAG_DEBUG_PTH_NS, J90 GND-IN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

Commit message: v22 production panel
Parts:
- U12, U19, U26, U33, U40, U8: value SN74AHC1G125 -> 74AHC1G125W5-7
- Y1, Y2, Y3, Y4, Y5, Y6: device SparkFun-Clocks:CRYSTAL-OSC-SMD-5X3 -> SparkFun-Clocks:CRYSTAL-SMD-3.2X2.5MM_GEYER_12.60421
- moved E$3 4.32 mm to (229.8, 149.9)
- moved E$4 4.32 mm to (229.8, 149.9)
- moved C158 0.85 mm to (198.3, 22.2)
- moved C65 0.85 mm to (119.0, 22.2)
- moved C7 0.85 mm to (39.8, 22.2)
- moved C236 0.85 mm to (39.8, 96.4)
- moved C314 0.85 mm to (119.0, 96.4)
- moved C392 0.85 mm to (198.3, 96.4)
- moved C9 0.72 mm to (39.0, 28.6)
- moved C64 0.72 mm to (118.2, 28.6)
- moved C235 0.72 mm to (39.0, 102.7)
- moved C157 0.72 mm to (197.5, 28.6)
- moved C313 0.72 mm to (118.2, 102.7)
- moved C391 0.72 mm to (197.5, 102.7)
Routing:
- net N$99: track 10.0 -> 8.21 mm
- net N$10: track 10.0 -> 8.21 mm
- net N$246: track 10.0 -> 8.21 mm
- net N$1: track 10.0 -> 8.21 mm
- net N$197: track 10.0 -> 8.21 mm
- net N$148: track 10.0 -> 8.21 mm
- net N$2: track 6.94 -> 6.21 mm
- net N$13: track 6.94 -> 6.21 mm
- net N$149: track 6.94 -> 6.21 mm
- net N$100: track 6.94 -> 6.21 mm
- net N$198: track 6.94 -> 6.21 mm
- net N$247: track 6.94 -> 6.21 mm
Other:
- board size 257.3 x 169.4 mm -> 261.1 x 168.4 mm
- board text added: "V22"
- board text removed: "V21"
