File: Hardware/Production/SparkFun_Tsunami_Qwiic-Panel.brd (EAGLE design)
At the start: 261.1 x 168.4 mm, 1956 parts, among them J1 VDC-IN, J10 TRIG2, J11 TRIG1, J12 3.3VA, J14 AUDIO I/O, J15 MIDI, J16 USB-C, J17 AGND, J19 3.3V, J2 GND-IN, J20 TRIG2, J21 TRIG1, J22 MIDI, J23 DEBUG, J24 PLAYING, J25 VDC-IN, J26 GND-IN, J27 USB-C, J28 QWIIC, J29 AGND, J3 DEBUG, J32 CORTEX_JTAG_DEBUG_PTH_NS, J33 AUDIO I/O, J34 3.3VA, J35 3.3V, J36 TRIG2, J37 TRIG1, J38 MIDI, J39 DEBUG, J4 QWIIC, J40 PLAYING, J41 VDC-IN, J42 GND-IN, J43 USB-C, J44 QWIIC, J45 AGND, J48 CORTEX_JTAG_DEBUG_PTH_NS, J49 AUDIO I/O, J5 AUDIO I/O, J50 3.3VA, J51 3.3V, J52 TRIG2, J53 TRIG1, J54 MIDI, J55 DEBUG, J56 PLAYING, J57 VDC-IN, J58 GND-IN, J59 USB-C, J6 3.3VA, J60 QWIIC, J61 AGND, J64 CORTEX_JTAG_DEBUG_PTH_NS, J65 AUDIO I/O, J66 3.3VA, J67 3.3V, J68 TRIG2, J69 TRIG1, J7 3.3V, J70 MIDI, J71 DEBUG, J72 PLAYING, J73 VDC-IN, J74 GND-IN, J75 USB-C, J76 QWIIC, J77 AGND, J8 PLAYING, J80 CORTEX_JTAG_DEBUG_PTH_NS, J81 AUDIO I/O, J82 3.3VA, J83 3.3V, J84 TRIG2, J85 TRIG1, J86 MIDI, J87 DEBUG, J88 PLAYING, J89 VDC-IN, J9 CORTEX_JTAG_DEBUG_PTH_NS, J90 GND-IN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

Commit message: v23 production panel
Parts:
- TP1, TP10, TP11, TP12, TP13, TP14, TP15, TP16, TP17, TP18, TP19, TP2, TP20, TP21, TP22, TP23, TP24, TP25, TP26, TP27, TP28, TP29, TP3, TP30, TP31, TP32, TP33, TP34, TP35, TP36, TP37, TP38, TP39, TP4, TP40, TP41, TP42, TP43, TP44, TP45, TP46, TP47, TP48, TP5, TP6, TP7, TP8, TP9: device SparkFun-Connectors:TP_15TH -> SparkFun-Connectors:PAD.03X.05
- flipped TP1 to the bottom
- flipped TP10 to the bottom
- flipped TP11 to the bottom
- flipped TP12 to the bottom
- flipped TP13 to the bottom
- flipped TP14 to the bottom
- flipped TP15 to the bottom
- flipped TP16 to the bottom
- flipped TP17 to the bottom
- flipped TP18 to the bottom
- flipped TP19 to the bottom
- flipped TP2 to the bottom
- flipped TP20 to the bottom
- flipped TP21 to the bottom
- flipped TP22 to the bottom
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Routing:
- net I2C_SDA1: track 30.7 -> 31.1 mm, vias 1 -> 2
- net I2C_SDA5: track 30.7 -> 31.1 mm, vias 1 -> 2
- net I2C_SDA4: track 30.7 -> 31.1 mm, vias 1 -> 2
- net I2C_SDA: track 30.7 -> 31.1 mm, vias 1 -> 2
- net I2C_SDA3: track 30.7 -> 31.1 mm, vias 1 -> 2
- net I2C_SDA2: track 30.7 -> 31.1 mm, vias 1 -> 2
- net I2C_SCK3: track 42.6 -> 42.9 mm, vias 1 -> 2
- net I2C_SCK5: track 42.6 -> 42.9 mm, vias 1 -> 2
- net SWDIO/TMS: track 20.8 -> 21.0 mm, vias 1 -> 2
- net I2C_SCK4: track 42.6 -> 42.9 mm, vias 1 -> 2
- net I2C_SCK2: track 42.6 -> 42.9 mm, vias 1 -> 2
- net I2C_SCK1: track 42.6 -> 42.9 mm, vias 1 -> 2
- net I2C_SCK: track 42.6 -> 42.9 mm, vias 1 -> 2
- net SWDIO/TMS1: track 20.8 -> 21.0 mm, vias 1 -> 2
- net SWDIO/TMS3: track 20.8 -> 21.0 mm, vias 1 -> 2
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Other:
- board text added: "V23"
- board text removed: "V22"
